File: samd21g_breakout.kicad_pcb (KiCad board)
At the start: 2 copper layers, 26.4 x 49.3 mm, 17 parts, among them J1 Conn_01x19, J2 Conn_01x19, J3 USB_B_Micro, U1 ATSAMD21G18A-AU, U2 MIC5504-3.3YM5, Y1 32768Hz

Commit message: update to kicad 6 format
Other:
- net class Default removed
